Commit message: retargeting

File: rby1_dg5f.urdf (robot description, URDF)
Before this commit: robot RBY1_UB, 76 links, 75 joints
Links:
- link base: geometry visual mesh filename=rby1/rby1ub_src/urdf/meshes/UB_LINK_BASE.dae
- link left_hand_ll_dg_1_1: geometry collision mesh filename=dg5f/meshes/dg5f_left/collision/ll_dg_1_1_c.STL; visual mesh filename=dg5f/meshes/dg5f_left/visual/ll_dg_1_1.dae
- link left_hand_ll_dg_1_2: geometry collision mesh filename=dg5f/meshes/dg5f_left/collision/ll_dg_1_2_c.STL; visual mesh filename=dg5f/meshes/dg5f_left/visual/ll_dg_1_2.dae
- link left_hand_ll_dg_1_3: geometry collision mesh filename=dg5f/meshes/dg5f_left/collision/ll_dg_1_3_c.STL; visual mesh filename=dg5f/meshes/dg5f_left/visual/ll_dg_1_3.dae
- link left_hand_ll_dg_1_4: geometry collision mesh filename=dg5f/meshes/dg5f_left/collision/ll_dg_1_4_c.STL; visual mesh filename=dg5f/meshes/dg5f_left/visual/ll_dg_1_4.dae
- link left_hand_ll_dg_1_tip: geometry collision mesh filename=dg5f/meshes/dg5f_left/collision/ll_dg_1_tip_c.STL; visual mesh filename=dg5f/meshes/dg5f_left/visual/ll_dg_1_tip.dae
- link left_hand_ll_dg_2_1: geometry collision mesh filename=dg5f/meshes/dg5f_left/collision/ll_dg_2_1_c.STL; visual mesh filename=dg5f/meshes/dg5f_left/visual/ll_dg_2_1.dae
- link left_hand_ll_dg_2_2: geometry collision mesh filename=dg5f/meshes/dg5f_left/collision/ll_dg_2_2_c.STL; visual mesh filename=dg5f/meshes/dg5f_left/visual/ll_dg_2_2.dae
- link left_hand_ll_dg_2_3: geometry collision mesh filename=dg5f/meshes/dg5f_left/collision/ll_dg_2_3_c.STL; visual mesh filename=dg5f/meshes/dg5f_left/visual/ll_dg_2_3.dae
- link left_hand_ll_dg_2_4: geometry collision mesh filename=dg5f/meshes/dg5f_left/collision/ll_dg_2_4_c.STL; visual mesh filename=dg5f/meshes/dg5f_left/visual/ll_dg_2_4.dae
- link left_hand_ll_dg_2_tip: geometry collision mesh filename=dg5f/meshes/dg5f_left/collision/ll_dg_2_tip_c.STL; visual mesh filename=dg5f/meshes/dg5f_left/visual/ll_dg_2_tip.dae
- link left_hand_ll_dg_3_1: geometry collision mesh filename=dg5f/meshes/dg5f_left/collision/ll_dg_3_1_c.STL; visual mesh filename=dg5f/meshes/dg5f_left/visual/ll_dg_3_1.dae
- link left_hand_ll_dg_3_2: geometry collision mesh filename=dg5f/meshes/dg5f_left/collision/ll_dg_3_2_c.STL; visual mesh filename=dg5f/meshes/dg5f_left/visual/ll_dg_3_2.dae
- link left_hand_ll_dg_3_3: geometry collision mesh filename=dg5f/meshes/dg5f_left/collision/ll_dg_3_3_c.STL; visual mesh filename=dg5f/meshes/dg5f_left/visual/ll_dg_3_3.dae
- link left_hand_ll_dg_3_4: geometry collision mesh filename=dg5f/meshes/dg5f_left/collision/ll_dg_3_4_c.STL; visual mesh filename=dg5f/meshes/dg5f_left/visual/ll_dg_3_4.dae
- link left_hand_ll_dg_3_tip: geometry collision mesh filename=dg5f/meshes/dg5f_left/collision/ll_dg_3_tip_c.STL; visual mesh filename=dg5f/meshes/dg5f_left/visual/ll_dg_3_tip.dae
- link left_hand_ll_dg_4_1: geometry collision mesh filename=dg5f/meshes/dg5f_left/collision/ll_dg_4_1_c.STL; visual mesh filename=dg5f/meshes/dg5f_left/visual/ll_dg_4_1.dae
- link left_hand_ll_dg_4_2: geometry collision mesh filename=dg5f/meshes/dg5f_left/collision/ll_dg_4_2_c.STL; visual mesh filename=dg5f/meshes/dg5f_left/visual/ll_dg_4_2.dae
- link left_hand_ll_dg_4_3: geometry collision mesh filename=dg5f/meshes/dg5f_left/collision/ll_dg_4_3_c.STL; visual mesh filename=dg5f/meshes/dg5f_left/visual/ll_dg_4_3.dae
- link left_hand_ll_dg_4_4: geometry collision mesh filename=dg5f/meshes/dg5f_left/collision/ll_dg_4_4_c.STL; visual mesh filename=dg5f/meshes/dg5f_left/visual/ll_dg_4_4.dae
- link left_hand_ll_dg_4_tip: geometry collision mesh filename=dg5f/meshes/dg5f_left/collision/ll_dg_4_tip_c.STL; visual mesh filename=dg5f/meshes/dg5f_left/visual/ll_dg_4_tip.dae
- link left_hand_ll_dg_5_1: geometry collision mesh filename=dg5f/meshes/dg5f_left/collision/ll_dg_5_1_c.STL; visual mesh filename=dg5f/meshes/dg5f_left/visual/ll_dg_5_1.dae
- link left_hand_ll_dg_5_2: geometry collision mesh filename=dg5f/meshes/dg5f_left/collision/ll_dg_5_2_c.STL; visual mesh filename=dg5f/meshes/dg5f_left/visual/ll_dg_5_2.dae
- link left_hand_ll_dg_5_3: geometry collision mesh filename=dg5f/meshes/dg5f_left/collision/ll_dg_5_3_c.STL; visual mesh filename=dg5f/meshes/dg5f_left/visual/ll_dg_5_3.dae
- link left_hand_ll_dg_5_4: geometry collision mesh filename=dg5f/meshes/dg5f_left/collision/ll_dg_5_4_c.STL; visual mesh filename=dg5f/meshes/dg5f_left/visual/ll_dg_5_4.dae
- link left_hand_ll_dg_5_tip: geometry collision mesh filename=dg5f/meshes/dg5f_left/collision/ll_dg_5_tip_c.STL; visual mesh filename=dg5f/meshes/dg5f_left/visual/ll_dg_5_tip.dae
- link left_hand_ll_dg_base: geometry collision mesh filename=dg5f/meshes/dg5f_left/collision/ll_dg_base_c.STL; visual mesh filename=dg5f/meshes/dg5f_left/visual/ll_dg_base.dae
- link left_hand_ll_dg_mount: geometry collision mesh filename=dg5f/meshes/dg5f_left/collision/ll_dg_mount_c.STL; visual mesh filename=dg5f/meshes/dg5f_left/visual/ll_dg_mount.dae
- link left_hand_ll_dg_palm: geometry collision mesh filename=dg5f/meshes/dg5f_left/collision/ll_dg_palm_c.STL; visual mesh filename=dg5f/meshes/dg5f_left/visual/ll_dg_palm.dae
- link link_head_0: geometry visual mesh filename=rby1/rby1ub_src/urdf/meshes/PAN_TILT_1.dae
- link link_head_1: geometry visual mesh filename=rby1/rby1ub_src/urdf/meshes/PAN_TILT_2.dae
- link link_head_2: geometry visual mesh filename=rby1/rby1ub_src/urdf/meshes/PAN_TILT_3.dae
- link link_left_arm_0: geometry collision capsule length=0.0700 radius=0.075; visual mesh filename=rby1/rby1ub_src/urdf/meshes/LINK_14.dae
- link link_left_arm_1: geometry collision capsule colaffinity=768 length=0.2000 radius=0.050; visual mesh filename=rby1/rby1ub_src/urdf/meshes/LINK_15.dae
- link link_left_arm_2: geometry collision capsule colaffinity=768 length=0.080000 radius=0.05; visual mesh filename=rby1/rby1ub_src/urdf/meshes/LINK_16.dae
- link link_left_arm_3: geometry collision capsule colaffinity=926 length=0.1150 radius=0.04; visual mesh filename=rby1/rby1ub_src/urdf/meshes/LINK_17.dae
- link link_left_arm_4: geometry collision capsule colaffinity=1022 length=0.095000 radius=0.035; visual mesh filename=rby1/rby1ub_src/urdf/meshes/LINK_18.dae
- link link_left_arm_5: geometry collision capsule colaffinity=1023 length=0.25 radius=0.075; visual mesh filename=rby1/rby1ub_src/urdf/meshes/LINK_19.dae
- link link_left_arm_6: geometry visual mesh filename=rby1/rby1ub_src/urdf/meshes/LINK_20.dae
- link link_right_arm_0: geometry collision capsule length=0.0700 radius=0.075; visual mesh filename=rby1/rby1ub_src/urdf/meshes/LINK_7.dae
- link link_right_arm_1: geometry collision capsule coltype=32 length=0.2 radius=0.05; visual mesh filename=rby1/rby1ub_src/urdf/meshes/LINK_8.dae
- link link_right_arm_2: geometry collision capsule coltype=64 length=0.080000 radius=0.05; visual mesh filename=rby1/rby1ub_src/urdf/meshes/LINK_9.dae
- link link_right_arm_3: geometry collision capsule colaffinity=30 coltype=128 length=0.1150 radius=0.04; visual mesh filename=rby1/rby1ub_src/urdf/meshes/LINK_10.dae
- link link_right_arm_4: geometry collision capsule colaffinity=30 coltype=256 length=0.095 radius=0.035; visual mesh filename=rby1/rby1ub_src/urdf/meshes/LINK_11.dae
- link link_right_arm_5: geometry collision capsule colaffinity=31 coltype=512 length=0.25 radius=0.075; visual mesh filename=rby1/rby1ub_src/urdf/meshes/LINK_12.dae
- link link_right_arm_6: geometry visual mesh filename=rby1/rby1ub_src/urdf/meshes/LINK_13.dae
- link link_torso_5: geometry collision capsule coltype=16 length=0.1350 radius=0.155; visual mesh filename=rby1/rby1ub_src/urdf/meshes/LINK_6.dae
- link link_torso_hp: geometry collision capsule coltype=8 length=0.2 radius=0.105; visual mesh filename=rby1/rby1ub_src/urdf/meshes/UB_LINK_HP.dae
- link right_hand_rl_dg_1_1: geometry collision mesh filename=dg5f/meshes/dg5f_right/collision/rl_dg_1_1_c.STL; visual mesh filename=dg5f/meshes/dg5f_right/visual/rl_dg_1_1.dae
- link right_hand_rl_dg_1_2: geometry collision mesh filename=dg5f/meshes/dg5f_right/collision/rl_dg_1_2_c.STL; visual mesh filename=dg5f/meshes/dg5f_right/visual/rl_dg_1_2.dae
- link right_hand_rl_dg_1_3: geometry collision mesh filename=dg5f/meshes/dg5f_right/collision/rl_dg_1_3_c.STL; visual mesh filename=dg5f/meshes/dg5f_right/visual/rl_dg_1_3.dae
- link right_hand_rl_dg_1_4: geometry collision mesh filename=dg5f/meshes/dg5f_right/collision/rl_dg_1_4_c.STL; visual mesh filename=dg5f/meshes/dg5f_right/visual/rl_dg_1_4.dae
- link right_hand_rl_dg_1_tip: geometry collision mesh filename=dg5f/meshes/dg5f_right/collision/rl_dg_1_tip_c.STL; visual mesh filename=dg5f/meshes/dg5f_right/visual/rl_dg_1_tip.dae
- link right_hand_rl_dg_2_1: geometry collision mesh filename=dg5f/meshes/dg5f_right/collision/rl_dg_2_1_c.STL; visual mesh filename=dg5f/meshes/dg5f_right/visual/rl_dg_2_1.dae
- link right_hand_rl_dg_2_2: geometry collision mesh filename=dg5f/meshes/dg5f_right/collision/rl_dg_2_2_c.STL; visual mesh filename=dg5f/meshes/dg5f_right/visual/rl_dg_2_2.dae
- link right_hand_rl_dg_2_3: geometry collision mesh filename=dg5f/meshes/dg5f_right/collision/rl_dg_2_3_c.STL; visual mesh filename=dg5f/meshes/dg5f_right/visual/rl_dg_2_3.dae
- link right_hand_rl_dg_2_4: geometry collision mesh filename=dg5f/meshes/dg5f_right/collision/rl_dg_2_4_c.STL; visual mesh filename=dg5f/meshes/dg5f_right/visual/rl_dg_2_4.dae
- link right_hand_rl_dg_2_tip: geometry collision mesh filename=dg5f/meshes/dg5f_right/collision/rl_dg_2_tip_c.STL; visual mesh filename=dg5f/meshes/dg5f_right/visual/rl_dg_2_tip.dae
- link right_hand_rl_dg_3_1: geometry collision mesh filename=dg5f/meshes/dg5f_right/collision/rl_dg_3_1_c.STL; visual mesh filename=dg5f/meshes/dg5f_right/visual/rl_dg_3_1.dae
- link right_hand_rl_dg_3_2: geometry collision mesh filename=dg5f/meshes/dg5f_right/collision/rl_dg_3_2_c.STL; visual mesh filename=dg5f/meshes/dg5f_right/visual/rl_dg_3_2.dae
- link right_hand_rl_dg_3_3: geometry collision mesh filename=dg5f/meshes/dg5f_right/collision/rl_dg_3_3_c.STL; visual mesh filename=dg5f/meshes/dg5f_right/visual/rl_dg_3_3.dae
- link right_hand_rl_dg_3_4: geometry collision mesh filename=dg5f/meshes/dg5f_right/collision/rl_dg_3_4_c.STL; visual mesh filename=dg5f/meshes/dg5f_right/visual/rl_dg_3_4.dae
- link right_hand_rl_dg_3_tip: geometry collision mesh filename=dg5f/meshes/dg5f_right/collision/rl_dg_3_tip_c.STL; visual mesh filename=dg5f/meshes/dg5f_right/visual/rl_dg_3_tip.dae
- link right_hand_rl_dg_4_1: geometry collision mesh filename=dg5f/meshes/dg5f_right/collision/rl_dg_4_1_c.STL; visual mesh filename=dg5f/meshes/dg5f_right/visual/rl_dg_4_1.dae
- link right_hand_rl_dg_4_2: geometry collision mesh filename=dg5f/meshes/dg5f_right/collision/rl_dg_4_2_c.STL; visual mesh filename=dg5f/meshes/dg5f_right/visual/rl_dg_4_2.dae
- link right_hand_rl_dg_4_3: geometry collision mesh filename=dg5f/meshes/dg5f_right/collision/rl_dg_4_3_c.STL; visual mesh filename=dg5f/meshes/dg5f_right/visual/rl_dg_4_3.dae
- link right_hand_rl_dg_4_4: geometry collision mesh filename=dg5f/meshes/dg5f_right/collision/rl_dg_4_4_c.STL; visual mesh filename=dg5f/meshes/dg5f_right/visual/rl_dg_4_4.dae
- link right_hand_rl_dg_4_tip: geometry collision mesh filename=dg5f/meshes/dg5f_right/collision/rl_dg_4_tip_c.STL; visual mesh filename=dg5f/meshes/dg5f_right/visual/rl_dg_4_tip.dae
- link right_hand_rl_dg_5_1: geometry collision mesh filename=dg5f/meshes/dg5f_right/collision/rl_dg_5_1_c.STL; visual mesh filename=dg5f/meshes/dg5f_right/visual/rl_dg_5_1.dae
- link right_hand_rl_dg_5_2: geometry collision mesh filename=dg5f/meshes/dg5f_right/collision/rl_dg_5_2_c.STL; visual mesh filename=dg5f/meshes/dg5f_right/visual/rl_dg_5_2.dae
- link right_hand_rl_dg_5_3: geometry collision mesh filename=dg5f/meshes/dg5f_right/collision/rl_dg_5_3_c.STL; visual mesh filename=dg5f/meshes/dg5f_right/visual/rl_dg_5_3.dae
- link right_hand_rl_dg_5_4: geometry collision mesh filename=dg5f/meshes/dg5f_right/collision/rl_dg_5_4_c.STL; visual mesh filename=dg5f/meshes/dg5f_right/visual/rl_dg_5_4.dae
- link right_hand_rl_dg_5_tip: geometry collision mesh filename=dg5f/meshes/dg5f_right/collision/rl_dg_5_tip_c.STL; visual mesh filename=dg5f/meshes/dg5f_right/visual/rl_dg_5_tip.dae
- link right_hand_rl_dg_base: geometry collision mesh filename=dg5f/meshes/dg5f_right/collision/rl_dg_base_c.STL; visual mesh filename=dg5f/meshes/dg5f_right/visual/rl_dg_base.dae
- link right_hand_rl_dg_mount: geometry collision mesh filename=dg5f/meshes/dg5f_right/collision/rl_dg_mount_c.STL; visual mesh filename=dg5f/meshes/dg5f_right/visual/rl_dg_mount.dae
- link right_hand_rl_dg_palm: geometry collision mesh filename=dg5f/meshes/dg5f_right/collision/rl_dg_palm_c.STL; visual mesh filename=dg5f/meshes/dg5f_right/visual/rl_dg_palm.dae
Joints:
- joint left_hand_mount: origin xyz=0.0 0.0 -0.1548 rpy=3.14159265358979 0.0 0.0 -> xyz=0.0 0.0 -0.1087 rpy=3.14159265358979 0.0 0.0
- joint right_hand_mount: origin xyz=0.0 0.0 -0.1548 rpy=3.14159265358979 0.0 0.0 -> xyz=0.0 0.0 -0.1087 rpy=3.14159265358979 0.0 0.0

File: robot_hand/urdf/dg5f_left.urdf (robot description, URDF)
Before this commit: robot dg5f_left_hand, 28 links, 27 joints
Links:
- link left_hand_ll_dg_1_1: geometry collision capsule length=0.041950 radius=0.010313; collision mesh filename=../dg5f/meshes/dg5f_left/collision/ll_dg_1_1_c.STL
- link left_hand_ll_dg_1_2: geometry collision capsule length=0.031000 radius=0.011669; collision mesh filename=../dg5f/meshes/dg5f_left/collision/ll_dg_1_2_c.STL
- link left_hand_ll_dg_1_3: geometry collision capsule length=0.038800 radius=0.011449; collision mesh filename=../dg5f/meshes/dg5f_left/collision/ll_dg_1_3_c.STL
- link left_hand_ll_dg_1_4: geometry collision capsule length=0.036300 radius=0.011558; collision mesh filename=../dg5f/meshes/dg5f_left/collision/ll_dg_1_4_c.STL
- link left_hand_ll_dg_2_1: geometry collision capsule length=0.031840 radius=0.012798; collision mesh filename=../dg5f/meshes/dg5f_left/collision/ll_dg_2_1_c.STL
- link left_hand_ll_dg_2_2: geometry collision capsule length=0.038800 radius=0.011449; collision mesh filename=../dg5f/meshes/dg5f_left/collision/ll_dg_2_2_c.STL
- link left_hand_ll_dg_2_3: geometry collision capsule length=0.038800 radius=0.011449; collision mesh filename=../dg5f/meshes/dg5f_left/collision/ll_dg_2_3_c.STL
- link left_hand_ll_dg_2_4: geometry collision capsule length=0.025500 radius=0.011517; collision mesh filename=../dg5f/meshes/dg5f_left/collision/ll_dg_2_4_c.STL
- link left_hand_ll_dg_3_1: geometry collision capsule length=0.031840 radius=0.013173; collision mesh filename=../dg5f/meshes/dg5f_left/collision/ll_dg_3_1_c.STL
- link left_hand_ll_dg_3_2: geometry collision capsule length=0.038800 radius=0.011449; collision mesh filename=../dg5f/meshes/dg5f_left/collision/ll_dg_3_2_c.STL
- link left_hand_ll_dg_3_3: geometry collision capsule length=0.038800 radius=0.011449; collision mesh filename=../dg5f/meshes/dg5f_left/collision/ll_dg_3_3_c.STL
- link left_hand_ll_dg_3_4: geometry collision capsule length=0.025500 radius=0.011517; collision mesh filename=../dg5f/meshes/dg5f_left/collision/ll_dg_3_4_c.STL
- link left_hand_ll_dg_4_1: geometry collision capsule length=0.031840 radius=0.012780; collision mesh filename=../dg5f/meshes/dg5f_left/collision/ll_dg_4_1_c.STL
- link left_hand_ll_dg_4_2: geometry collision capsule length=0.038800 radius=0.011449; collision mesh filename=../dg5f/meshes/dg5f_left/collision/ll_dg_4_2_c.STL
- link left_hand_ll_dg_4_3: geometry collision capsule length=0.038800 radius=0.011449; collision mesh filename=../dg5f/meshes/dg5f_left/collision/ll_dg_4_3_c.STL
- link left_hand_ll_dg_4_4: geometry collision capsule length=0.025500 radius=0.011517; collision mesh filename=../dg5f/meshes/dg5f_left/collision/ll_dg_4_4_c.STL
- link left_hand_ll_dg_5_1: geometry collision capsule length=0.047282 radius=0.012988; collision mesh filename=../dg5f/meshes/dg5f_left/collision/ll_dg_5_1_c.STL
- link left_hand_ll_dg_5_2: geometry collision capsule length=0.031000 radius=0.011669; collision mesh filename=../dg5f/meshes/dg5f_left/collision/ll_dg_5_2_c.STL
- link left_hand_ll_dg_5_3: geometry collision capsule length=0.038800 radius=0.011449; collision mesh filename=../dg5f/meshes/dg5f_left/collision/ll_dg_5_3_c.STL
- link left_hand_ll_dg_5_4: geometry collision capsule length=0.036300 radius=0.011558; collision mesh filename=../dg5f/meshes/dg5f_left/collision/ll_dg_5_4_c.STL

File: robot_hand/urdf/dg5f_right.urdf (robot description, URDF)
Before this commit: robot dg5f_right_hand, 28 links, 27 joints
Links:
- link right_hand_rl_dg_1_1: geometry collision capsule length=0.041950 radius=0.010313; collision mesh filename=../dg5f/meshes/dg5f_right/collision/rl_dg_1_1_c.STL
- link right_hand_rl_dg_1_2: geometry collision capsule length=0.031000 radius=0.011669; collision mesh filename=../dg5f/meshes/dg5f_right/collision/rl_dg_1_2_c.STL
- link right_hand_rl_dg_1_3: geometry collision capsule length=0.038800 radius=0.011449; collision mesh filename=../dg5f/meshes/dg5f_right/collision/rl_dg_1_3_c.STL
- link right_hand_rl_dg_1_4: geometry collision capsule length=0.036300 radius=0.011558; collision mesh filename=../dg5f/meshes/dg5f_right/collision/rl_dg_1_4_c.STL
- link right_hand_rl_dg_2_1: geometry collision capsule length=0.031840 radius=0.012780; collision mesh filename=../dg5f/meshes/dg5f_right/collision/rl_dg_2_1_c.STL
- link right_hand_rl_dg_2_2: geometry collision capsule length=0.038800 radius=0.011449; collision mesh filename=../dg5f/meshes/dg5f_right/collision/rl_dg_2_2_c.STL
- link right_hand_rl_dg_2_3: geometry collision capsule length=0.038800 radius=0.011449; collision mesh filename=../dg5f/meshes/dg5f_right/collision/rl_dg_2_3_c.STL
- link right_hand_rl_dg_2_4: geometry collision capsule length=0.025500 radius=0.011517; collision mesh filename=../dg5f/meshes/dg5f_right/collision/rl_dg_2_4_c.STL
- link right_hand_rl_dg_3_1: geometry collision capsule length=0.031840 radius=0.013182; collision mesh filename=../dg5f/meshes/dg5f_right/collision/rl_dg_3_1_c.STL
- link right_hand_rl_dg_3_2: geometry collision capsule length=0.038800 radius=0.011449; collision mesh filename=../dg5f/meshes/dg5f_right/collision/rl_dg_3_2_c.STL
- link right_hand_rl_dg_3_3: geometry collision capsule length=0.038800 radius=0.011449; collision mesh filename=../dg5f/meshes/dg5f_right/collision/rl_dg_3_3_c.STL
- link right_hand_rl_dg_3_4: geometry collision capsule length=0.025500 radius=0.011517; collision mesh filename=../dg5f/meshes/dg5f_right/collision/rl_dg_3_4_c.STL
- link right_hand_rl_dg_4_1: geometry collision capsule length=0.031840 radius=0.012794; collision mesh filename=../dg5f/meshes/dg5f_right/collision/rl_dg_4_1_c.STL
- link right_hand_rl_dg_4_2: geometry collision capsule length=0.038800 radius=0.011449; collision mesh filename=../dg5f/meshes/dg5f_right/collision/rl_dg_4_2_c.STL
- link right_hand_rl_dg_4_3: geometry collision capsule length=0.038800 radius=0.011449; collision mesh filename=../dg5f/meshes/dg5f_right/collision/rl_dg_4_3_c.STL
- link right_hand_rl_dg_4_4: geometry collision capsule length=0.025500 radius=0.011517; collision mesh filename=../dg5f/meshes/dg5f_right/collision/rl_dg_4_4_c.STL
- link right_hand_rl_dg_5_1: geometry collision capsule length=0.047282 radius=0.013359; collision mesh filename=../dg5f/meshes/dg5f_right/collision/rl_dg_5_1_c.STL
- link right_hand_rl_dg_5_2: geometry collision capsule length=0.031000 radius=0.011669; collision mesh filename=../dg5f/meshes/dg5f_right/collision/rl_dg_5_2_c.STL
- link right_hand_rl_dg_5_3: geometry collision capsule length=0.038800 radius=0.011449; collision mesh filename=../dg5f/meshes/dg5f_right/collision/rl_dg_5_3_c.STL
- link right_hand_rl_dg_5_4: geometry collision capsule length=0.036300 radius=0.011558; collision mesh filename=../dg5f/meshes/dg5f_right/collision/rl_dg_5_4_c.STL

Commit message: teaching data generation, camera pose should be fixed

File: rby1_dg5f.urdf (robot description, URDF)
Before this commit: robot RBY1_UB, 76 links, 75 joints
Links:
- link link_head_2: geometry visual box size=0.03 0.04 0.024; visual mesh filename=rby1/rby1ub_src/urdf/meshes/PAN_TILT_3.dae
- link link_left_arm_6: geometry visual box size=0.03 0.04 0.024; visual mesh filename=rby1/rby1ub_src/urdf/meshes/LINK_20.dae
- link link_right_arm_6: geometry visual box size=0.03 0.04 0.024; visual mesh filename=rby1/rby1ub_src/urdf/meshes/LINK_13.dae

Commit message: rendering thread decomposition

File: rby1_dg5f.urdf (robot description, URDF)
Before this commit: robot RBY1_UB, 76 links, 75 joints
Links:
- link link_left_arm_6: geometry visual box size=0.024 0.04 0.03; visual mesh filename=rby1/rby1ub_src/urdf/meshes/LINK_20.dae
- link link_right_arm_6: geometry visual box size=0.024 0.04 0.03; visual mesh filename=rby1/rby1ub_src/urdf/meshes/LINK_13.dae

Commit message: benchmarking hand retarget (pinch grip doesnt work ㅠㅠ)

File: rby1_dg5f.urdf (robot description, URDF)
Before this commit: robot RBY1_UB, 76 links, 75 joints
Joints:
- joint left_arm_2: limit lower=-3.141592654 upper=3.141592654 effort=70.0 velocity=3.141592654 -> lower=-1.570796327 upper=0 effort=70.0 velocity=3.141592654
- joint left_arm_4: limit lower=-3.141592654 upper=3.141592654 effort=10.0 velocity=6.283185308 -> lower=-1.570796327 upper=1.570796327 effort=10.0 velocity=6.283185308
- joint left_arm_6: limit lower=-2.705260340 upper=2.705260340 effort=8.0 velocity=2.094395102 -> lower=-2.705260340 upper=0 effort=8.0 velocity=2.094395102
- joint right_arm_2: limit lower=-3.141592654 upper=3.141592654 effort=70.0 velocity=3.141592654 -> lower=0 upper=1.570796327 effort=70.0 velocity=3.141592654
- joint right_arm_4: limit lower=-3.141592654 upper=3.141592654 effort=10.0 velocity=6.283185308 -> lower=-1.570796327 upper=1.570796327 effort=10.0 velocity=6.283185308
- joint right_arm_6: limit lower=-2.705260340 upper=2.705260340 effort=8.0 velocity=2.094395102 -> lower=0 upper=2.705260340 effort=8.0 velocity=2.094395102
